File: kicad/RadioExercise/RadioExercise.sch (KiCad schematic (older format))
At the start: 14 parts

Commit message: update
Parts:
- removed TP? (x2): TestPoint, symbol Connector:TestPoint
- added D?: LED, symbol Device:LED
- added R?: R, symbol Device:R
Connections:
- net GND: now also D?.1 (K)
- net VDD: now also IC?.3 (WP#/SIO2)
- net at IC?.14 (RC3): now also IC?.5 (~CE)
- net at IC?.22 (RB1): now also IC?.1 (CE#)
- net at IC?.23 (RB2): now also IC?.6 (SCK)
- net at IC?.24 (RB3): now also IC?.2 (SO/SIO1)
- net at IC?.25 (RB4): now also IC?.5 (SI/SIO0)
- net at IC?.26 (RB5): now also R?.2
- net at IC?.1 (OUTN): now also LS?.1
- net at IC?.7 (OUTP): now also LS?.2
- new net: D?.2 (A), R?.1
Other:
- moved on the sheet: C?, IC?, LS?

Commit message: change
Parts:
- removed C? (x2): C, symbol Device:C
- removed TP? (x2): TestPoint, symbol Connector:TestPoint
- added C3, C5: 10u, Capacitor_THT:CP_Radial_D4.0mm_P1.50mm, symbol Device:CP
- added J1: Conn_01x02_Female, symbol Connector:Conn_01x02_Female
- added R1, R2, R3, R5: 10k, symbol Device:R
- added SW1, SW2, SW3, SW4: SW_MEC_5E, symbol Switch:SW_MEC_5E
- added SW5: SW_DPDT_x2, symbol Switch:SW_DPDT_x2
- C1: renamed from C?; value C -> 1u; footprint (none) -> Capacitor_THT:C_Disc_D7.5mm_W5.0mm_P5.00mm
- C2: renamed from C?; value CP -> 47u; footprint (none) -> Capacitor_THT:CP_Radial_D4.0mm_P1.50mm
- C4: value C -> 1u; footprint (none) -> Capacitor_THT:C_Disc_D7.5mm_W5.0mm_P5.00mm
- D1: renamed from D?; footprint (none) -> LED_THT:LED_D5.0mm_Clear
- IC1: renamed from IC?; footprint SOIC127P600X175-8N -> Package_DIP:DIP-8_W7.62mm
- IC2: renamed from IC?; footprint DIP794W56P254L3486H508Q28N -> PIC16F1778-I_SP:DIP794W56P254L3486H508Q28N
- IC3: renamed from IC?; footprint SOIC127P794X203-8N -> SST26VF064B-104I_SM:SOIC127P794X203-8N
- R4: renamed from R?; value R -> 15k
- gave numbers to parts that had none: 2
Connections:
- net GND: now also C3.2, C5.2, J1.1 (Pin_1), R1.2, R2.2, R3.2, SW4.3 (K)
- net VDD: now also C3.1, C5.1, R5.1, SW1.1, SW2.1, SW3.1, SW5.2 (B)
- net at IC2.1 (VPP/~MCLR~/RE3): now also R5.2, SW4.2
- net at IC2.11 (RC0): now also R1.1, SW1.4 (A)
- net at IC2.12 (RC1): now also R2.1, SW2.4 (A)
- net at IC2.13 (RC2): now also R3.1, SW3.4 (A)
- new net: J1.2 (Pin_2), SW5.3 (C)
- no-connect marks 0 -> 23
Other:
- moved on the sheet: R4

Commit message: update
Parts:
- J1, LS1: footprint (none) -> RadioExercise:Conn_01x02_SMD
- R1, R2, R3, R4, R5: footprint (none) -> Resistor_THT:R_Axial_DIN0207_L6.3mm_D2.5mm_P7.62mm_Horizontal
- R6: value R -> 1k; footprint (none) -> Resistor_THT:R_Axial_DIN0207_L6.3mm_D2.5mm_P7.62mm_Horizontal
- SW1, SW2, SW3, SW4: footprint (none) -> Button_Switch_THT:SW_PUSH_6mm
- SW5: footprint (none) -> RadioExercise:SW_slide_01x03_THT
Changed lines of the file:
@@
 F 0 "R4" V 3893 3100 50  0000 C CNN
 F 1 "15k" V 3984 3100 50  0000 C CNN
-F 2 "" V 4030 3100 50  0001 C CNN
+F 2 "Resistor_THT:R_Axial_DIN0207_L6.3mm_D2.5mm_P7.62mm_Horizontal" V 4030 3100 50  0001 C CNN
 F 3 "~" H 4100 3100 50  0001 C CNN
 	1    4100 3100
@@
 F 0 "LS1" V 2959 1620 50  0000 R CNN
 F 1 "Speaker" V 2868 1620 50  0000 R CNN
-F 2 "" H 2950 1700 50  0001 C CNN
+F 2 "RadioExercise:Conn_01x02_SMD" H 2950 1700 50  0001 C CNN
 F 3 "~" H 2940 1850 50  0001 C CNN
 	1    2950 1900
@@
 F 0 "J1" H 4392 5025 50  0000 C CNN
 F 1 "Conn_01x02_Female" H 4392 5116 50  0000 C CNN
-F 2 "" H 4500 5350 50  0001 C CNN
+F 2 "RadioExercise:Conn_01x02_SMD" H 4500 5350 50  0001 C CNN
 F 3 "~" H 4500 5350 50  0001 C CNN
 	1    4500 5350
@@
 F 0 "SW5" H 5050 4525 50  0000 C CNN
 F 1 "SW_DPDT_x2" H 5050 4616 50  0000 C CNN
-F 2 "" H 5050 4850 50  0001 C CNN
+F 2 "RadioExercise:SW_slide_01x03_THT" H 5050 4850 50  0001 C CNN
 F 3 "~" H 5050 4850 50  0001 C CNN
 	1    5050 4850
@@
 F 0 "SW4" H 4750 2535 50  0000 C CNN
 F 1 "SW_MEC_5E" H 4750 2444 50  0000 C CNN
-F 2 "" H 4750 2450 50  0001 C CNN
+F 2 "Button_Switch_THT:SW_PUSH_6mm" H 4750 2450 50  0001 C CNN
 F 3 "http://www.apem.com/int/index.php?controller=attachment&id_attachment=1371" H 4750 2450 50  0001 C CNN
 	1    4750 2150
@@
 F 0 "SW1" H 2950 5185 50  0000 C CNN
 F 1 "SW_MEC_5E" H 2950 5094 50  0000 C CNN
-F 2 "" H 2950 5100 50  0001 C CNN
+F 2 "Button_Switch_THT:SW_PUSH_6mm" H 2950 5100 50  0001 C CNN
 F 3 "http://www.apem.com/int/index.php?controller=attachment&id_attachment=1371" H 2950 5100 50  0001 C CNN
 	1    2950 4800
@@
 F 0 "SW2" H 2950 5735 50  0000 C CNN
 F 1 "SW_MEC_5E" H 2950 5644 50  0000 C CNN
-F 2 "" H 2950 5650 50  0001 C CNN
+F 2 "Button_Switch_THT:SW_PUSH_6mm" H 2950 5650 50  0001 C CNN
 F 3 "http://www.apem.com/int/index.php?controller=attachment&id_attachment=1371" H 2950 5650 50  0001 C CNN
 	1    2950 5350
@@
 F 0 "SW3" H 2950 6335 50  0000 C CNN
 F 1 "SW_MEC_5E" H 2950 6244 50  0000 C CNN
-F 2 "" H 2950 6250 50  0001 C CNN
+F 2 "Button_Switch_THT:SW_PUSH_6mm" H 2950 6250 50  0001 C CNN
 F 3 "http://www.apem.com/int/index.php?controller=attachment&id_attachment=1371" H 2950 6250 50  0001 C CNN
 	1    2950 5950
@@
 F 0 "R5" H 4420 2696 50  0000 L CNN
 F 1 "10k" H 4420 2605 50  0000 L CNN
-F 2 "" V 4280 2650 50  0001 C CNN
+F 2 "Resistor_THT:R_Axial_DIN0207_L6.3mm_D2.5mm_P7.62mm_Horizontal" V 4280 2650 50  0001 C CNN
 F 3 "~" H 4350 2650 50  0001 C CNN
 	1    4350 2650
@@
 F 0 "R1" H 3670 4646 50  0000 L CNN
 F 1 "10k" H 3670 4555 50  0000 L CNN
-F 2 "" V 3530 4600 50  0001 C CNN
+F 2 "Resistor_THT:R_Axial_DIN0207_L6.3mm_D2.5mm_P7.62mm_Horizontal" V 3530 4600 50  0001 C CNN
 F 3 "~" H 3600 4600 50  0001 C CNN
 	1    3600 4600
@@
 F 0 "R2" H 3970 5246 50  0000 L CNN
 F 1 "10k" H 3970 5155 50  0000 L CNN
-F 2 "" V 3830 5200 50  0001 C CNN
+F 2 "Resistor_THT:R_Axial_DIN0207_L6.3mm_D2.5mm_P7.62mm_Horizontal" V 3830 5200 50  0001 C CNN
 F 3 "~" H 3900 5200 50  0001 C CNN
 	1    3900 5200
@@
 P 6700 2250
 F 0 "R6" H 6770 2296 50  0000 L CNN
-F 1 "R" H 6770 2205 50  0000 L CNN
-F 2 "" V 6630 2250 50  0001 C CNN
+F 1 "1k" H 6770 2205 50  0000 L CNN
+F 2 "Resistor_THT:R_Axial_DIN0207_L6.3mm_D2.5mm_P7.62mm_Horizontal" V 6630 2250 50  0001 C CNN
 F 3 "~" H 6700 2250 50  0001 C CNN
 	1    6700 2250
@@
 F 0 "R3" H 4120 5896 50  0000 L CNN
 F 1 "10k" H 4120 5805 50  0000 L CNN
-F 2 "" V 3980 5850 50  0001 C CNN
+F 2 "Resistor_THT:R_Axial_DIN0207_L6.3mm_D2.5mm_P7.62mm_Horizontal" V 3980 5850 50  0001 C CNN
 F 3 "~" H 4050 5850 50  0001 C CNN
 	1    4050 5850

Commit message: update
Parts:
- removed D1: LED, LED_THT:LED_D5.0mm_Clear, symbol Device:LED
- removed R1: 10k, Resistor_THT:R_Axial_DIN0207_L6.3mm_D2.5mm_P7.62mm_Horizontal, symbol Device:R
- removed R6: 1k, Resistor_THT:R_Axial_DIN0207_L6.3mm_D2.5mm_P7.62mm_Horizontal, symbol Device:R
- removed SW1, SW2, SW3, SW4: SW_MEC_5E, Button_Switch_THT:SW_PUSH_6mm, symbol Switch:SW_MEC_5E
- added SW1, SW2: SW_Push, Button_Switch_THT:SW_PUSH_6mm, symbol Switch:SW_Push
Connections:
- net GND: now also IC2.11 (RC0)
- net VDD: now also SW1.1, SW2.1
- net at IC2.12 (RC1), R2.1: now also SW1.2
- net at IC2.13 (RC2), R3.1: now also SW2.2
- no-connect marks 23 -> 16
Changed lines of the file:
@@
 Wire Wire Line
 	3050 2400 3050 2100
-$Comp
-L Device:LED D1
-U 1 1 607923B2
-P 6500 1650
-F 0 "D1" H 6493 1867 50  0000 C CNN
-F 1 "LED" H 6493 1776 50  0000 C CNN
-F 2 "LED_THT:LED_D5.0mm_Clear" H 6500 1650 50  0001 C CNN
-F 3 "~" H 6500 1650 50  0001 C CNN
-	1    6500 1650
-	1    0    0    -1
-$EndComp
-Wire Wire Line
-	6350 1650 6100 1650
-Wire Wire Line
-	6100 1650 6100 1900
-$Comp
-L power:GND #PWR016
-U 1 1 60797571
-P 6100 1900
-F 0 "#PWR016" H 6100 1650 50  0001 C CNN
-F 1 "GND" H 6105 1727 50  0000 C CNN
-F 2 "" H 6100 1900 50  0001 C CNN
-F 3 "" H 6100 1900 50  0001 C CNN
-	1    6100 1900
-	1    0    0    -1
-$EndComp
-Wire Wire Line
-	6600 3100 6700 3100
-Wire Wire Line
-	6700 1650 6650 1650
-Wire Wire Line
-	6700 2100 6700 1650
-Wire Wire Line
-	6700 3100 6700 2400
 Wire Wire Line
 	4700 4200 3400 4200
@@
 	4700 4750 4700 5250
 $Comp
-L Switch:SW_MEC_5E SW4
-U 1 1 607C8A2B
-P 4750 2150
-F 0 "SW4" H 4750 2535 50  0000 C CNN
-F 1 "SW_MEC_5E" H 4750 2444 50  0000 C CNN
-F 2 "Button_Switch_THT:SW_PUSH_6mm" H 4750 2450 50  0001 C CNN
-F 3 "http://www.apem.com/int/index.php?controller=attachment&id_attachment=1371" H 4750 2450 50  0001 C CNN
-	1    4750 2150
-	1    0    0    -1
-$EndComp
-$Comp
-L Switch:SW_MEC_5E SW1
-U 1 1 607CBCFF
-P 2950 4800
-F 0 "SW1" H 2950 5185 50  0000 C CNN
-F 1 "SW_MEC_5E" H 2950 5094 50  0000 C CNN
-F 2 "Button_Switch_THT:SW_PUSH_6mm" H 2950 5100 50  0001 C CNN
-F 3 "http://www.apem.com/int/index.php?controller=attachment&id_attachment=1371" H 2950 5100 50  0001 C CNN
-	1    2950 4800
-	1    0    0    -1
-$EndComp
-$Comp
-L Switch:SW_MEC_5E SW2
-U 1 1 607CCCF1
-P 2950 5350
-F 0 "SW2" H 2950 5735 50  0000 C CNN
-F 1 "SW_MEC_5E" H 2950 5644 50  0000 C CNN
-F 2 "Button_Switch_THT:SW_PUSH_6mm" H 2950 5650 50  0001 C CNN
-F 3 "http://www.apem.com/int/index.php?controller=attachment&id_attachment=1371" H 2950 5650 50  0001 C CNN
-	1    2950 5350
-	1    0    0    -1
-$EndComp
-$Comp
-L Switch:SW_MEC_5E SW3
-U 1 1 607CD3C9
-P 2950 5950
-F 0 "SW3" H 2950 6335 50  0000 C CNN
-F 1 "SW_MEC_5E" H 2950 6244 50  0000 C CNN
-F 2 "Button_Switch_THT:SW_PUSH_6mm" H 2950 6250 50  0001 C CNN
-F 3 "http://www.apem.com/int/index.php?controller=attachment&id_attachment=1371" H 2950 6250 50  0001 C CNN
-	1    2950 5950
-	1    0    0    -1
-$EndComp
-$Comp
 L power:VDD #PWR011
 U 1 1 607CDF26
@@
 $EndComp
 $Comp
-L power:GND #PWR014
-U 1 1 607CF093
-P 5100 2350
-F 0 "#PWR014" H 5100 2100 50  0001 C CNN
-F 1 "GND" H 5105 2177 50  0000 C CNN
-F 2 "" H 5100 2350 50  0001 C CNN
-F 3 "" H 5100 2350 50  0001 C CNN
-	1    5100 2350
-	1    0    0    -1
-$EndComp
-$Comp
 L Device:R R5
 U 1 1 607CFC46
@@
 Wire Wire Line
 	4350 2900 4350 2800
-Wire Wire Line
-	4700 2900 4550 2900
-Wire Wire Line
-	4550 2150 4550 2900
-Connection ~ 4550 2900
-Wire Wire Line
-	4550 2900 4350 2900
-Wire Wire Line
-	4950 2150 5100 2150
-Wire Wire Line
-	5100 2150 5100 2350
 $Comp
 L power:GND #PWR08
 U 1 1 607D61A2
-P 3600 4750
-F 0 "#PWR08" H 3600 4500 50  0001 C CNN
-F 1 "GND" H 3605 4577 50  0000 C CNN
-F 2 "" H 3600 4750 50  0001 C CNN
-F 3 "" H 3600 4750 50  0001 C CNN
-	1    3600 4750
-	1    0    0    -1
-$EndComp
-$Comp
-L Device:R R1
-U 1 1 607D795D
-P 3600 4600
-F 0 "R1" H 3670 4646 50  0000 L CNN
-F 1 "10k" H 3670 4555 50  0000 L CNN
-F 2 "Resistor_THT:R_Axial_DIN0207_L6.3mm_D2.5mm_P7.62mm_Horizontal" V 3530 4600 50  0001 C CNN
-F 3 "~" H 3600 4600 50  0001 C CNN
-	1    3600 4600
-	1    0    0    -1
-$EndComp
-$Comp
-L power:GND #PWR09
-U 1 1 607DBAD5
-P 3900 5350
-F 0 "#PWR09" H 3900 5100 50  0001 C CNN
-F 1 "GND" H 3905 5177 50  0000 C CNN
-F 2 "" H 3900 5350 50  0001 C CNN
-F 3 "" H 3900 5350 50  0001 C CNN
-	1    3900 5350
-	1    0    0    -1
-$EndComp
-$Comp
-L Device:R R2
-U 1 1 607DBADB
-P 3900 5200
-F 0 "R2" H 3970 5246 50  0000 L CNN
-F 1 "10k" H 3970 5155 50  0000 L CNN
-F 2 "Resistor_THT:R_Axial_DIN0207_L6.3mm_D2.5mm_P7.62mm_Horizontal" V 3830 5200 50  0001 C CNN
-F 3 "~" H 3900 5200 50  0001 C CNN
-	1    3900 5200
-	1    0    0    -1
-$EndComp
-$Comp
-L power:GND #PWR010
-U 1 1 607DCD73
-P 4050 6000
-F 0 "#PWR010" H 4050 5750 50  0001 C CNN
-F 1 "GND" H 4055 5827 50  0000 C CNN
-F 2 "" H 4050 6000 50  0001 C CNN
-F 3 "" H 4050 6000 50  0001 C CNN
-	1    4050 6000
-	1    0    0    -1
-$EndComp
-Wire Wire Line
-	4700 3900 3600 3900
-Wire Wire Line
-	3600 3900 3600 4350
-Wire Wire Line
-	4700 4000 3900 4000
-Wire Wire Line
-	3900 4000 3900 4950
+P 3600 3950
+F 0 "#PWR08" H 3600 3700 50  0001 C CNN
+F 1 "GND" H 3605 3777 50  0000 C CNN
+F 2 "" H 3600 3950 50  0001 C CNN
+F 3 "" H 3600 3950 50  0001 C CNN
+	1    3600 3950
+	1    0    0    -1
+$EndComp
 Wire Wire Line
 	4700 4100 4050 4100
-Wire Wire Line
-	4050 4100 4050 5650
-$Comp
-L power:VDD #PWR03
-U 1 1 607E225E
-P 2500 4700
-F 0 "#PWR03" H 2500 4550 50  0001 C CNN
-F 1 "VDD" H 2515 4873 50  0000 C CNN
-F 2 "" H 2500 4700 50  0001 C CNN
-F 3 "" H 2500 4700 50  0001 C CNN
-	1    2500 4700
-	1    0    0    -1
-$EndComp
-$Comp
-L power:VDD #PWR04
-U 1 1 607E3268
-P 2500 5250
-F 0 "#PWR04" H 2500 5100 50  0001 C CNN
-F 1 "VDD" H 2515 5423 50  0000 C CNN
-F 2 "" H 2500 5250 50  0001 C CNN
-F 3 "" H 2500 5250 50  0001 C CNN
-	1    2500 5250
-	1    0    0    -1
-$EndComp
-$Comp
-L power:VDD #PWR05
-U 1 1 607E39FD
-P 2500 5850
-F 0 "#PWR05" H 2500 5700 50  0001 C CNN
-F 1 "VDD" H 2515 6023 50  0000 C CNN
-F 2 "" H 2500 5850 50  0001 C CNN
-F 3 "" H 2500 5850 50  0001 C CNN
-	1    2500 5850
-	1    0    0    -1
-$EndComp
-Wire Wire Line
-	2750 4700 2500 4700
-Wire Wire Line
-	2750 5250 2500 5250
-Wire Wire Line
-	2750 5850 2500 5850
-Wire Wire Line
-	3600 4350 3150 4350
-Wire Wire Line
-	3150 4350 3150 4700
-Connection ~ 3600 4350
-Wire Wire Line
-	3600 4350 3600 4450
-Wire Wire Line
-	3900 4950 3250 4950
-Wire Wire Line
-	3250 4950 3250 5250
-Wire Wire Line
-	3250 5250 3150 5250
-Connection ~ 3900 4950
-Wire Wire Line
-	3900 4950 3900 5050
-Wire Wire Line
-	3250 5650 3250 5850
-Wire Wire Line
-	3250 5850 3150 5850
-Connection ~ 4050 5650
-Wire Wire Line
-	4050 5650 4050 5700
-Wire Wire Line
-	4050 5650 3250 5650
 NoConn ~ 4850 4950
-NoConn ~ 3150 4800
-NoConn ~ 2750 4800
-NoConn ~ 2750 5350
-NoConn ~ 3150 5350
-NoConn ~ 3150 5950
-NoConn ~ 2750 5950
 NoConn ~ 6600 4200
 NoConn ~ 6600 4100
@@
 NoConn ~ 4700 3700
 NoConn ~ 4700 3800
-NoConn ~ 4950 2050
-NoConn ~ 4550 2050
 Connection ~ 3400 3050
 Wire Wire Line
@@
 	0    1    1    0
 $EndComp
-$Comp
-L Device:R R6
-U 1 1 607980DD
-P 6700 2250
-F 0 "R6" H 6770 2296 50  0000 L CNN
-F 1 "1k" H 6770 2205 50  0000 L CNN
-F 2 "Resistor_THT:R_Axial_DIN0207_L6.3mm_D2.5mm_P7.62mm_Horizontal" V 6630 2250 50  0001 C CNN
-F 3 "~" H 6700 2250 50  0001 C CNN
-	1    6700 2250
-	1    0    0    -1
-$EndComp
+NoConn ~ 6600 3100
+Wire Wire Line
+	4350 2900 4700 2900
+Wire Wire Line
+	3600 3900 3600 3950
+Wire Wire Line
+	4700 4000 3900 4000
+Wire Wire Line
+	4700 3900 3600 3900
 $Comp
 L Device:R R3
@@
 	1    0    0    -1
 $EndComp
+Wire Wire Line
+	4050 5650 3250 5650
+Wire Wire Line
+	4050 5650 4050 5700
+Connection ~ 4050 5650
+Wire Wire Line
+	3250 5850 3150 5850
+Wire Wire Line
+	3250 5650 3250 5850
+Wire Wire Line
+	3900 4950 3900 5050
+Connection ~ 3900 4950
+Wire Wire Line
+	3250 5250 3150 5250
+Wire Wire Line
+	3250 4950 3250 5250
+Wire Wire Line
+	3900 4950 3250 4950
+Wire Wire Line
+	2750 5850 2500 5850
+Wire Wire Line
+	2750 5250 2500 5250
+$Comp
+L power:VDD #PWR05
+U 1 1 607E39FD
+P 2500 5850
+F 0 "#PWR05" H 2500 5700 50  0001 C CNN
+F 1 "VDD" H 2515 6023 50  0000 C CNN
+F 2 "" H 2500 5850 50  0001 C CNN
+F 3 "" H 2500 5850 50  0001 C CNN
+	1    2500 5850
+	1    0    0    -1
+$EndComp
+$Comp
+L power:VDD #PWR04
+U 1 1 607E3268
+P 2500 5250
+F 0 "#PWR04" H 2500 5100 50  0001 C CNN
+F 1 "VDD" H 2515 5423 50  0000 C CNN
+F 2 "" H 2500 5250 50  0001 C CNN
+F 3 "" H 2500 5250 50  0001 C CNN
+	1    2500 5250
+	1    0    0    -1
+$EndComp
+Wire Wire Line
+	4050 4100 4050 5650
+Wire Wire Line
+	3900 4000 3900 4950
+$Comp
+L power:GND #PWR010
+U 1 1 607DCD73
+P 4050 6000
+F 0 "#PWR010" H 4050 5750 50  0001 C CNN
+F 1 "GND" H 4055 5827 50  0000 C CNN
+F 2 "" H 4050 6000 50  0001 C CNN
+F 3 "" H 4050 6000 50  0001 C CNN
+	1    4050 6000
+	1    0    0    -1
+$EndComp
+$Comp
+L Device:R R2
+U 1 1 607DBADB
+P 3900 5200
+F 0 "R2" H 3970 5246 50  0000 L CNN
+F 1 "10k" H 3970 5155 50  0000 L CNN
+F 2 "Resistor_THT:R_Axial_DIN0207_L6.3mm_D2.5mm_P7.62mm_Horizontal" V 3830 5200 50  0001 C CNN
+F 3 "~" H 3900 5200 50  0001 C CNN
+	1    3900 5200
+	1    0    0    -1
+$EndComp
+$Comp
+L power:GND #PWR09
+U 1 1 607DBAD5
+P 3900 5350
+F 0 "#PWR09" H 3900 5100 50  0001 C CNN
+F 1 "GND" H 3905 5177 50  0000 C CNN
+F 2 "" H 3900 5350 50  0001 C CNN
+F 3 "" H 3900 5350 50  0001 C CNN
+	1    3900 5350
+	1    0    0    -1
+$EndComp
+$Comp
+L Switch:SW_Push SW1
+U 1 1 60798E1C
+P 2950 5250
+F 0 "SW1" H 2950 5535 50  0000 C CNN
+F 1 "SW_Push" H 2950 5444 50  0000 C CNN
+F 2 "Button_Switch_THT:SW_PUSH_6mm" H 2950 5450 50  0001 C CNN
+F 3 "~" H 2950 5450 50  0001 C CNN
+	1    2950 5250
+	1    0    0    -1
+$EndComp
+$Comp
+L Switch:SW_Push SW2
+U 1 1 6079D3D1
+P 2950 5850
+F 0 "SW2" H 2950 6135 50  0000 C CNN
+F 1 "SW_Push" H 2950 6044 50  0000 C CNN
+F 2 "Button_Switch_THT:SW_PUSH_6mm" H 2950 6050 50  0001 C CNN
+F 3 "~" H 2950 6050 50  0001 C CNN
+	1    2950 5850
+	1    0    0    -1
+$EndComp
