File: kicad/RadioExercise/music_writer/RadioExercise.sch (KiCad schematic (older format))
At the start: 24 parts, among them IC1 HT82V739, IC2 PIC16F1778-I_SP, IC3 SST26VF064B-104I_SM, J1 Conn_01x02_Female, SW1 SW_Push, SW2 SW_Push, SW5 SW_DPDT_x2

Commit message: change
Parts:
- IC1: symbol HT82V739:HT82V739 -> RadioExercise-rescue:HT82V739-HT82V739
- IC2: symbol PIC16F1778-I_SP:PIC16F1778-I_SP -> RadioExercise-rescue:PIC16F1778-I_SP-PIC16F1778-I_SP
- IC3: symbol SST26VF064B-104I_SM:SST26VF064B-104I_SM -> RadioExercise-rescue:SST26VF064B-104I_SM-SST26VF064B-104I_SM
- J1, LS1: footprint RadioExercise:Conn_01x02_SMD -> music_writer:conn_1x2
- SW5: footprint RadioExercise:SW_slide_01x03_THT -> music_writer:SW_slide
Connections:
- net GND: now also C5.2; no longer C5.1
- net VDD: now also C5.1; no longer C5.2
Changed lines of the file:
@@
 	2200 3350 2500 3350
 $Comp
-L HT82V739:HT82V739 IC1
+L RadioExercise-rescue:HT82V739-HT82V739 IC1
 U 1 1 6076049A
 P 2500 3250
@@
 F 0 "LS1" V 3259 1820 50  0000 R CNN
 F 1 "Speaker" V 3168 1820 50  0000 R CNN
-F 2 "RadioExercise:Conn_01x02_SMD" H 3250 1900 50  0001 C CNN
+F 2 "music_writer:conn_1x2" H 3250 1900 50  0001 C CNN
 F 3 "~" H 3240 2050 50  0001 C CNN
 	1    3250 2100
@@
 	7500 4200 7500 4000
 $Comp
-L PIC16F1778-I_SP:PIC16F1778-I_SP IC2
+L RadioExercise-rescue:PIC16F1778-I_SP-PIC16F1778-I_SP IC2
 U 1 1 6075AE19
 P 5000 3100
@@
 	9600 2950 9450 2950
 $Comp
-L SST26VF064B-104I_SM:SST26VF064B-104I_SM IC3
+L RadioExercise-rescue:SST26VF064B-104I_SM-SST26VF064B-104I_SM IC3
 U 1 1 6076184C
 P 7850 2750
@@
 F 0 "J1" H 4692 5225 50  0000 C CNN
 F 1 "Conn_01x02_Female" H 4692 5316 50  0000 C CNN
-F 2 "RadioExercise:Conn_01x02_SMD" H 4800 5550 50  0001 C CNN
+F 2 "music_writer:conn_1x2" H 4800 5550 50  0001 C CNN
 F 3 "~" H 4800 5550 50  0001 C CNN
 	1    4800 5550
@@
 F 0 "SW5" H 5350 4725 50  0000 C CNN
 F 1 "SW_DPDT_x2" H 5350 4816 50  0000 C CNN
-F 2 "RadioExercise:SW_slide_01x03_THT" H 5350 5050 50  0001 C CNN
+F 2 "music_writer:SW_slide" H 5350 5050 50  0001 C CNN
 F 3 "~" H 5350 5050 50  0001 C CNN
 	1    5350 5050
@@
 U 1 1 608606DE
 P 9700 2500
-F 0 "C5" H 9818 2546 50  0000 L CNN
-F 1 "10u" H 9818 2455 50  0000 L CNN
+F 0 "C5" V 9850 2450 50  0000 L CNN
+F 1 "10u" V 9550 2450 50  0000 L CNN
 F 2 "Capacitor_THT:CP_Radial_D4.0mm_P1.50mm" H 9738 2350 50  0001 C CNN
 F 3 "~" H 9700 2500 50  0001 C CNN
 	1    9700 2500
-	0    1    1    0
-$EndComp
-Wire Wire Line
+	0    -1   -1   0
+$EndComp
+Wire Wire Line
